Commit message: update path

File: franka_panda/urdf/panda.urdf (robot description, URDF)
Before this commit: robot panda, 13 links, 12 joints
Links:
- link panda_hand: geometry collision mesh filename=../meshes/collision/hand.stl; visual mesh filename=../meshes/visual/hand.dae
- link panda_leftfinger: geometry collision box size=17.5e-3 15.2e-3 18.5e-3; collision box size=17.5e-3 7e-3 23.5e-3
- link panda_link0: geometry collision mesh filename=../meshes/collision/link0.stl; visual mesh filename=../meshes/visual/link0.dae
- link panda_link1: geometry collision mesh filename=../meshes/collision/link1.stl; visual mesh filename=../meshes/visual/link1.dae
- link panda_link2: geometry collision mesh filename=../meshes/collision/link2.stl; visual mesh filename=../meshes/visual/link2.dae
- link panda_link3: geometry collision mesh filename=../meshes/collision/link3.stl; visual mesh filename=../meshes/visual/link3.dae
- link panda_link4: geometry collision mesh filename=../meshes/collision/link4.stl; visual mesh filename=../meshes/visual/link4.dae
- link panda_link5: geometry collision mesh filename=../meshes/collision/link5.stl; visual mesh filename=../meshes/visual/link5.dae
- link panda_link6: geometry collision mesh filename=../meshes/collision/link6.stl; visual mesh filename=../meshes/visual/link6.dae
- link panda_link7: geometry collision mesh filename=../meshes/collision/link7.stl; visual mesh filename=../meshes/visual/link7.dae
- link panda_rightfinger: geometry collision box size=17.5e-3 15.2e-3 18.5e-3; collision box size=17.5e-3 7e-3 23.5e-3

File: jaka_zu12/urdf/jaka.urdf (robot description, URDF)
Before this commit: robot jaka_zu12, 8 links, 7 joints
Links:
- link Link_0: geometry collision mesh filename=../assets/base_link.STL; visual mesh filename=../assets/base_link.STL
- link Link_1: geometry collision mesh filename=../assets/1.STL; visual mesh filename=../assets/1.STL
- link Link_2: geometry collision mesh filename=../assets/2.STL; visual mesh filename=../assets/2.STL
- link Link_3: geometry collision mesh filename=../assets/3.STL; visual mesh filename=../assets/3.STL
- link Link_4: geometry collision mesh filename=../assets/4.STL; visual mesh filename=../assets/4.STL
- link Link_5: geometry collision mesh filename=../assets/5.STL; visual mesh filename=../assets/5.STL
- link Link_6: geometry collision mesh filename=../assets/6.STL; visual mesh filename=../assets/6.STL

File: kinect_dk/urdf/azure_kinect_macro.urdf.xacro (robot description, xacro)
@@ -17,5 +17,5 @@
         <origin xyz="0 0 0" rpy="0 0 0" />
         <geometry>
-          <mesh filename="./assets/visual.dae"/>
+          <mesh filename="../assets/visual.dae"/>
         </geometry>
       </visual>
@@ -23,5 +23,5 @@
         <origin xyz="0 0 0" rpy="0 0 0" />
         <geometry>
-          <mesh filename="./assets/collision.stl"/>
+          <mesh filename="../assets/collision.stl"/>
         </geometry>
       </collision>

File: leap_hand/urdf/leap_hand_left.urdf (robot description, URDF)
Before this commit: robot leap_left, 22 links, 21 joints
Links:
- link dip: geometry collision box size=0.014 0.02 0.004; collision box size=0.014 0.02 0.004
- link dip_2: geometry collision box size=0.014 0.02 0.004; collision box size=0.014 0.02 0.004
- link dip_3: geometry collision box size=0.014 0.02 0.004; collision box size=0.014 0.02 0.004
- link fingertip: geometry collision box size=0.014 0.022 0.004; collision box size=0.014 0.022 0.004
- link fingertip_2: geometry collision box size=0.014 0.022 0.004; collision box size=0.014 0.022 0.004
- link fingertip_3: geometry collision box size=0.014 0.022 0.004; collision box size=0.014 0.022 0.004
- link mcp_joint: geometry collision box size=0.014 0.02 0.004; collision box size=0.014 0.02 0.004
- link mcp_joint_2: geometry collision box size=0.014 0.02 0.004; collision box size=0.014 0.02 0.004
- link mcp_joint_3: geometry collision box size=0.014 0.02 0.004; collision box size=0.014 0.02 0.004
- link palm_lower_left: geometry collision box size=0.004 0.036 0.034; collision box size=0.01 0.12 0.02
- link pip: geometry collision box size=0.034 0.026 0.022; visual mesh filename=../meshes/visual/pip.obj
- link pip_2: geometry collision box size=0.034 0.026 0.022; visual mesh filename=../meshes/visual/pip.obj
- link pip_3: geometry collision box size=0.034 0.026 0.022; visual mesh filename=../meshes/visual/pip.obj
- link thumb_dip: geometry collision box size=0.01 0.024 0.018; collision box size=0.014 0.02 0.004
- link thumb_fingertip: geometry collision box size=0.008 0.024 0.018; collision box size=0.02 0.004 0.03
- link thumb_left_temp_base: geometry collision box size=0.034 0.026 0.022; visual mesh filename=../meshes/visual/pip_left.obj
- link thumb_pip: geometry collision box size=0.014 0.004 0.02; collision box size=0.014 0.004 0.02

File: leap_hand/urdf/leap_hand_left_glb.urdf (robot description, URDF)
Before this commit: robot leap_left, 22 links, 21 joints
Links:
- link dip: geometry collision box size=0.014 0.02 0.004; collision box size=0.014 0.02 0.004
- link dip_2: geometry collision box size=0.014 0.02 0.004; collision box size=0.014 0.02 0.004
- link dip_3: geometry collision box size=0.014 0.02 0.004; collision box size=0.014 0.02 0.004
- link fingertip: geometry collision box size=0.014 0.022 0.004; collision box size=0.014 0.022 0.004
- link fingertip_2: geometry collision box size=0.014 0.022 0.004; collision box size=0.014 0.022 0.004
- link fingertip_3: geometry collision box size=0.014 0.022 0.004; collision box size=0.014 0.022 0.004
- link mcp_joint: geometry collision box size=0.014 0.02 0.004; collision box size=0.014 0.02 0.004
- link mcp_joint_2: geometry collision box size=0.014 0.02 0.004; collision box size=0.014 0.02 0.004
- link mcp_joint_3: geometry collision box size=0.014 0.02 0.004; collision box size=0.014 0.02 0.004
- link palm_lower_left: geometry collision box size=0.004 0.036 0.034; collision box size=0.01 0.12 0.02
- link pip: geometry collision box size=0.034 0.026 0.022; visual mesh filename=../meshes/visual/pip.glb
- link pip_2: geometry collision box size=0.034 0.026 0.022; visual mesh filename=../meshes/visual/pip.glb
- link pip_3: geometry collision box size=0.034 0.026 0.022; visual mesh filename=../meshes/visual/pip.glb
- link thumb_dip: geometry collision box size=0.01 0.024 0.018; collision box size=0.014 0.02 0.004
- link thumb_fingertip: geometry collision box size=0.008 0.024 0.018; collision box size=0.02 0.004 0.03
- link thumb_left_temp_base: geometry collision box size=0.034 0.026 0.022; visual mesh filename=../meshes/visual/pip_left.glb
- link thumb_pip: geometry collision box size=0.014 0.004 0.02; collision box size=0.014 0.004 0.02

File: leap_hand/urdf/leap_hand_right.urdf (robot description, URDF)
Before this commit: robot leap_right, 22 links, 21 joints
Links:
- link dip: geometry collision box size=0.014 0.02 0.004; collision box size=0.014 0.02 0.004
- link dip_2: geometry collision box size=0.014 0.02 0.004; collision box size=0.014 0.02 0.004
- link dip_3: geometry collision box size=0.014 0.02 0.004; collision box size=0.014 0.02 0.004
- link fingertip: geometry collision box size=0.014 0.022 0.004; collision box size=0.014 0.022 0.004
- link fingertip_2: geometry collision box size=0.014 0.022 0.004; collision box size=0.014 0.022 0.004
- link fingertip_3: geometry collision box size=0.014 0.022 0.004; collision box size=0.014 0.022 0.004
- link mcp_joint: geometry collision box size=0.014 0.02 0.004; collision box size=0.014 0.02 0.004
- link mcp_joint_2: geometry collision box size=0.014 0.02 0.004; collision box size=0.014 0.02 0.004
- link mcp_joint_3: geometry collision box size=0.014 0.02 0.004; collision box size=0.014 0.02 0.004
- link palm_lower: geometry collision box size=0.004 0.036 0.034; collision box size=0.01 0.12 0.02
- link pip: geometry collision box size=0.034 0.026 0.022; visual mesh filename=../meshes/visual/pip.obj
- link pip_2: geometry collision box size=0.034 0.026 0.022; visual mesh filename=../meshes/visual/pip.obj
- link pip_3: geometry collision box size=0.034 0.026 0.022; visual mesh filename=../meshes/visual/pip.obj
- link thumb_dip: geometry collision box size=0.01 0.024 0.018; collision box size=0.014 0.02 0.004
- link thumb_fingertip: geometry collision box size=0.008 0.024 0.018; collision box size=0.02 0.004 0.03
- link thumb_pip: geometry collision box size=0.014 0.004 0.02; collision box size=0.014 0.004 0.02
- link thumb_temp_base: geometry collision box size=0.034 0.026 0.022; visual mesh filename=../meshes/visual/pip.obj

File: leap_hand/urdf/leap_hand_right_glb.urdf (robot description, URDF)
Before this commit: robot leap_right, 22 links, 21 joints
Links:
- link dip: geometry collision box size=0.014 0.02 0.004; collision box size=0.014 0.02 0.004
- link dip_2: geometry collision box size=0.014 0.02 0.004; collision box size=0.014 0.02 0.004
- link dip_3: geometry collision box size=0.014 0.02 0.004; collision box size=0.014 0.02 0.004
- link fingertip: geometry collision box size=0.014 0.022 0.004; collision box size=0.014 0.022 0.004
- link fingertip_2: geometry collision box size=0.014 0.022 0.004; collision box size=0.014 0.022 0.004
- link fingertip_3: geometry collision box size=0.014 0.022 0.004; collision box size=0.014 0.022 0.004
- link mcp_joint: geometry collision box size=0.014 0.02 0.004; collision box size=0.014 0.02 0.004
- link mcp_joint_2: geometry collision box size=0.014 0.02 0.004; collision box size=0.014 0.02 0.004
- link mcp_joint_3: geometry collision box size=0.014 0.02 0.004; collision box size=0.014 0.02 0.004
- link palm_lower: geometry collision box size=0.004 0.036 0.034; collision box size=0.01 0.12 0.02
- link pip: geometry collision box size=0.034 0.026 0.022; visual mesh filename=../meshes/visual/pip.glb
- link pip_2: geometry collision box size=0.034 0.026 0.022; visual mesh filename=../meshes/visual/pip.glb
- link pip_3: geometry collision box size=0.034 0.026 0.022; visual mesh filename=../meshes/visual/pip.glb
- link thumb_dip: geometry collision box size=0.01 0.024 0.018; collision box size=0.014 0.02 0.004
- link thumb_fingertip: geometry collision box size=0.008 0.024 0.018; collision box size=0.02 0.004 0.03
- link thumb_pip: geometry collision box size=0.014 0.004 0.02; collision box size=0.014 0.004 0.02
- link thumb_temp_base: geometry collision box size=0.034 0.026 0.022; visual mesh filename=../meshes/visual/pip.glb

File: ur10/urdf/ur10.urdf (robot description, URDF)
Before this commit: robot ur10_robot, 11 links, 10 joints
Links:
- link base_link_inertia: geometry collision mesh filename=../assets/base.stl; visual mesh filename=../assets/base.dae
- link forearm_link: geometry collision mesh filename=../assets/forearm.stl; visual mesh filename=../assets/forearm.dae
- link shoulder_link: geometry collision mesh filename=../assets/shoulder.stl; visual mesh filename=../assets/shoulder.dae
- link upper_arm_link: geometry collision mesh filename=../assets/upperarm.stl; visual mesh filename=../assets/upperarm.dae
- link wrist_1_link: geometry collision mesh filename=../assets/wrist1.stl; visual mesh filename=../assets/wrist1.dae
- link wrist_2_link: geometry collision mesh filename=../assets/wrist2.stl; visual mesh filename=../assets/wrist2.dae
- link wrist_3_link: geometry collision mesh filename=../assets/wrist3.stl; visual mesh filename=../assets/wrist3.dae
