Commit message: add dexrobot021 mimic property

File: dexrobot_021/urdf/dexhand021_left_simplified_mimic.urdf (robot description, URDF)
Before this commit: robot dexhand021_left_simplified, 26 links, 25 joints
Joints:
- joint l_f_joint1_4: mimic (none) -> joint=l_f_joint1_3 multiplier=1.0 offset=0.0
- joint l_f_joint2_4: mimic (none) -> joint=l_f_joint2_3 multiplier=1.0 offset=0.0
- joint l_f_joint3_1: axis 0 0 1 -> (none); limit lower=-0.001 upper=0.001 effort=10 velocity=1.5 -> (none); type revolute -> fixed
- joint l_f_joint3_4: mimic (none) -> joint=l_f_joint3_3 multiplier=1.0 offset=0.0
- joint l_f_joint4_4: mimic (none) -> joint=l_f_joint4_3 multiplier=1.0 offset=0.0
- joint l_f_joint5_4: mimic (none) -> joint=l_f_joint5_3 multiplier=1.0 offset=0.0

Commit message: update dexrobot021 params

File: dexrobot_021/urdf/dexhand021_left_simplified_mimic.urdf (robot description, URDF)
Before this commit: robot dexhand021_left_simplified, 26 links, 25 joints
Joints:
- joint l_f_joint1_3: mimic (none) -> joint=l_f_joint1_4 multiplier=1.0096 offset=0.0795
- joint l_f_joint1_4: mimic joint=l_f_joint1_3 multiplier=1.0 offset=0.0 -> (none)
- joint l_f_joint2_3: mimic (none) -> joint=l_f_joint2_4 multiplier=1.0096 offset=0.0795
- joint l_f_joint2_4: mimic joint=l_f_joint2_3 multiplier=1.0 offset=0.0 -> (none)
- joint l_f_joint3_3: mimic (none) -> joint=l_f_joint3_4 multiplier=1.0096 offset=0.0795
- joint l_f_joint3_4: mimic joint=l_f_joint3_3 multiplier=1.0 offset=0.0 -> (none)
- joint l_f_joint4_3: mimic (none) -> joint=l_f_joint4_4 multiplier=1.0096 offset=0.0795
- joint l_f_joint4_4: mimic joint=l_f_joint4_3 multiplier=1.0 offset=0.0 -> (none)
- joint l_f_joint5_1: limit lower=0 upper=0.632 effort=10 velocity=1.5 -> lower=0 upper=0.6 effort=10 velocity=1.5; mimic joint=l_f_joint2_1 multiplier=1.8162 offset=0.0180973190139292 -> joint=l_f_joint2_1 multiplier=1.8162 offset=0.0181
- joint l_f_joint5_3: mimic (none) -> joint=l_f_joint5_4 multiplier=1.0096 offset=0.0795
- joint l_f_joint5_4: mimic joint=l_f_joint5_3 multiplier=1.0 offset=0.0 -> (none)

File: dexrobot_021/urdf/dexhand021_right_simplified_mimic.urdf (robot description, URDF)
Before this commit: robot dexhand021_right_simplified_mimic, 26 links, 25 joints
Joints:
- joint r_f_joint1_3: mimic (none) -> joint=r_f_joint1_4 multiplier=1.0096 offset=0.0795
- joint r_f_joint1_4: mimic joint=r_f_joint1_3 multiplier=1.0 offset=0.0 -> (none)
- joint r_f_joint2_3: mimic (none) -> joint=r_f_joint2_4 multiplier=1.0096 offset=0.0795
- joint r_f_joint2_4: mimic joint=r_f_joint2_3 multiplier=1.0 offset=0.0 -> (none)
- joint r_f_joint3_3: mimic (none) -> joint=r_f_joint3_4 multiplier=1.0096 offset=0.0795
- joint r_f_joint3_4: mimic joint=r_f_joint3_3 multiplier=1.0 offset=0.0 -> (none)
- joint r_f_joint4_3: mimic (none) -> joint=r_f_joint4_4 multiplier=1.0096 offset=0.0795
- joint r_f_joint4_4: mimic joint=r_f_joint4_3 multiplier=1.0 offset=0.0 -> (none)
- joint r_f_joint5_1: limit lower=0 upper=0.632 effort=10 velocity=1.5 -> lower=0 upper=0.6 effort=10 velocity=1.5; mimic joint=r_f_joint2_1 multiplier=1.8162 offset=0.0180973190139292 -> joint=r_f_joint2_1 multiplier=1.8162 offset=0.0181
- joint r_f_joint5_3: mimic (none) -> joint=r_f_joint5_4 multiplier=1.0096 offset=0.0795
- joint r_f_joint5_4: mimic joint=r_f_joint5_3 multiplier=1.0 offset=0.0 -> (none)
