Commit message: DexHand 021: drive the PIP joint, let the DIP follow
The SDK's *_dip channel actuates and senses the PIP (Yuan et al. 2025 RA-L
Sec. II-C/D; protractor on the hardware 2026-09-15), but every mimic model
drove *_4 (DIP) and derived *_3 (PIP) from it.

- MJCF (left/right convex+primitive mimic, ur10_dexhand_inhand/grasp):
  actuators act_*_4 -> act_*_3 with unchanged parameters and order;
  equality now *_4 = g(*_3), g = 0.0001 + 0.6446x + 0.2340x^2 - 0.0631x^3
  + 0.0359x^4 fitted to 末端指节映射关系.csv (rms 0.004 deg); PIP range 0-1.3
  (firmware 74.7 deg cap), DIP range 0-1.2; drive/passive joint classes swapped.
  Fingertip positions match the old model at the same physical pose to 0.02 mm.
- URDF (same variants + scene/urdf/ur10_dexhand): <mimic> moved from *_3 to
  *_4, linear DIP = 0.9023 PIP - 0.0410 (max 3.7 deg vs the csv; the old
  PIP = f(DIP) line was 4.6 deg), DIP limit -0.05..1.2.
- USD mimic variants regenerated with tools/convert_urdfs_to_usd.py
  (PhysX mimic now on *_4 referencing *_3).

Co-Authored-By: Claude <noreply@anthropic.com>

File: dexrobot_021/urdf/dexhand021_left_convex_mimic.urdf (robot description, URDF)
Before this commit: robot dexhand021_left_convex_mimic, 26 links, 25 joints
Joints:
- joint l_f_joint1_3: mimic joint=l_f_joint1_4 multiplier=1.0096 offset=0.0795 -> (none)
- joint l_f_joint1_4: limit lower=0 upper=1.3 effort=10 velocity=1.5 -> lower=-0.05 upper=1.2 effort=10 velocity=1.5; mimic (none) -> joint=l_f_joint1_3 multiplier=0.9023 offset=-0.0410
- joint l_f_joint2_3: mimic joint=l_f_joint2_4 multiplier=1.0096 offset=0.0795 -> (none)
- joint l_f_joint2_4: limit lower=0 upper=1.3 effort=10 velocity=1.5 -> lower=-0.05 upper=1.2 effort=10 velocity=1.5; mimic (none) -> joint=l_f_joint2_3 multiplier=0.9023 offset=-0.0410
- joint l_f_joint3_3: mimic joint=l_f_joint3_4 multiplier=1.0096 offset=0.0795 -> (none)
- joint l_f_joint3_4: limit lower=0 upper=1.3 effort=10 velocity=1.5 -> lower=-0.05 upper=1.2 effort=10 velocity=1.5; mimic (none) -> joint=l_f_joint3_3 multiplier=0.9023 offset=-0.0410
- joint l_f_joint4_3: mimic joint=l_f_joint4_4 multiplier=1.0096 offset=0.0795 -> (none)
- joint l_f_joint4_4: limit lower=0 upper=1.3 effort=10 velocity=1.5 -> lower=-0.05 upper=1.2 effort=10 velocity=1.5; mimic (none) -> joint=l_f_joint4_3 multiplier=0.9023 offset=-0.0410
- joint l_f_joint5_3: mimic joint=l_f_joint5_4 multiplier=1.0096 offset=0.0795 -> (none)
- joint l_f_joint5_4: limit lower=0 upper=1.3 effort=10 velocity=1.5 -> lower=-0.05 upper=1.2 effort=10 velocity=1.5; mimic (none) -> joint=l_f_joint5_3 multiplier=0.9023 offset=-0.0410

File: dexrobot_021/urdf/dexhand021_left_primitive_mimic.urdf (robot description, URDF)
Before this commit: robot dexhand021_left_primitive_mimic, 26 links, 25 joints
Joints:
- joint l_f_joint1_3: mimic joint=l_f_joint1_4 multiplier=1.0096 offset=0.0795 -> (none)
- joint l_f_joint1_4: limit lower=0 upper=1.3 effort=10 velocity=1.5 -> lower=-0.05 upper=1.2 effort=10 velocity=1.5; mimic (none) -> joint=l_f_joint1_3 multiplier=0.9023 offset=-0.0410
- joint l_f_joint2_3: mimic joint=l_f_joint2_4 multiplier=1.0096 offset=0.0795 -> (none)
- joint l_f_joint2_4: limit lower=0 upper=1.3 effort=10 velocity=1.5 -> lower=-0.05 upper=1.2 effort=10 velocity=1.5; mimic (none) -> joint=l_f_joint2_3 multiplier=0.9023 offset=-0.0410
- joint l_f_joint3_3: mimic joint=l_f_joint3_4 multiplier=1.0096 offset=0.0795 -> (none)
- joint l_f_joint3_4: limit lower=0 upper=1.3 effort=10 velocity=1.5 -> lower=-0.05 upper=1.2 effort=10 velocity=1.5; mimic (none) -> joint=l_f_joint3_3 multiplier=0.9023 offset=-0.0410
- joint l_f_joint4_3: mimic joint=l_f_joint4_4 multiplier=1.0096 offset=0.0795 -> (none)
- joint l_f_joint4_4: limit lower=0 upper=1.3 effort=10 velocity=1.5 -> lower=-0.05 upper=1.2 effort=10 velocity=1.5; mimic (none) -> joint=l_f_joint4_3 multiplier=0.9023 offset=-0.0410
- joint l_f_joint5_3: mimic joint=l_f_joint5_4 multiplier=1.0096 offset=0.0795 -> (none)
- joint l_f_joint5_4: limit lower=0 upper=1.3 effort=10 velocity=1.5 -> lower=-0.05 upper=1.2 effort=10 velocity=1.5; mimic (none) -> joint=l_f_joint5_3 multiplier=0.9023 offset=-0.0410

File: dexrobot_021/urdf/dexhand021_right_convex_mimic.urdf (robot description, URDF)
Before this commit: robot dexhand021_right_convex_mimic, 26 links, 25 joints
Joints:
- joint r_f_joint1_3: mimic joint=r_f_joint1_4 multiplier=1.0096 offset=0.0795 -> (none)
- joint r_f_joint1_4: limit lower=0 upper=1.3 effort=10 velocity=1.5 -> lower=-0.05 upper=1.2 effort=10 velocity=1.5; mimic (none) -> joint=r_f_joint1_3 multiplier=0.9023 offset=-0.0410
- joint r_f_joint2_3: mimic joint=r_f_joint2_4 multiplier=1.0096 offset=0.0795 -> (none)
- joint r_f_joint2_4: limit lower=0 upper=1.3 effort=10 velocity=1.5 -> lower=-0.05 upper=1.2 effort=10 velocity=1.5; mimic (none) -> joint=r_f_joint2_3 multiplier=0.9023 offset=-0.0410
- joint r_f_joint3_3: mimic joint=r_f_joint3_4 multiplier=1.0096 offset=0.0795 -> (none)
- joint r_f_joint3_4: limit lower=0 upper=1.3 effort=10 velocity=1.5 -> lower=-0.05 upper=1.2 effort=10 velocity=1.5; mimic (none) -> joint=r_f_joint3_3 multiplier=0.9023 offset=-0.0410
- joint r_f_joint4_3: mimic joint=r_f_joint4_4 multiplier=1.0096 offset=0.0795 -> (none)
- joint r_f_joint4_4: limit lower=0 upper=1.3 effort=10 velocity=1.5 -> lower=-0.05 upper=1.2 effort=10 velocity=1.5; mimic (none) -> joint=r_f_joint4_3 multiplier=0.9023 offset=-0.0410
- joint r_f_joint5_3: mimic joint=r_f_joint5_4 multiplier=1.0096 offset=0.0795 -> (none)
- joint r_f_joint5_4: limit lower=0 upper=1.3 effort=10 velocity=1.5 -> lower=-0.05 upper=1.2 effort=10 velocity=1.5; mimic (none) -> joint=r_f_joint5_3 multiplier=0.9023 offset=-0.0410

File: dexrobot_021/urdf/dexhand021_right_primitive_mimic.urdf (robot description, URDF)
Before this commit: robot dexhand021_right_primitive_mimic, 26 links, 25 joints
Joints:
- joint r_f_joint1_3: mimic joint=r_f_joint1_4 multiplier=1.0096 offset=0.0795 -> (none)
- joint r_f_joint1_4: limit lower=0 upper=1.3 effort=10 velocity=1.5 -> lower=-0.05 upper=1.2 effort=10 velocity=1.5; mimic (none) -> joint=r_f_joint1_3 multiplier=0.9023 offset=-0.0410
- joint r_f_joint2_3: mimic joint=r_f_joint2_4 multiplier=1.0096 offset=0.0795 -> (none)
- joint r_f_joint2_4: limit lower=0 upper=1.3 effort=10 velocity=1.5 -> lower=-0.05 upper=1.2 effort=10 velocity=1.5; mimic (none) -> joint=r_f_joint2_3 multiplier=0.9023 offset=-0.0410
- joint r_f_joint3_3: mimic joint=r_f_joint3_4 multiplier=1.0096 offset=0.0795 -> (none)
- joint r_f_joint3_4: limit lower=0 upper=1.3 effort=10 velocity=1.5 -> lower=-0.05 upper=1.2 effort=10 velocity=1.5; mimic (none) -> joint=r_f_joint3_3 multiplier=0.9023 offset=-0.0410
- joint r_f_joint4_3: mimic joint=r_f_joint4_4 multiplier=1.0096 offset=0.0795 -> (none)
- joint r_f_joint4_4: limit lower=0 upper=1.3 effort=10 velocity=1.5 -> lower=-0.05 upper=1.2 effort=10 velocity=1.5; mimic (none) -> joint=r_f_joint4_3 multiplier=0.9023 offset=-0.0410
- joint r_f_joint5_3: mimic joint=r_f_joint5_4 multiplier=1.0096 offset=0.0795 -> (none)
- joint r_f_joint5_4: limit lower=0 upper=1.3 effort=10 velocity=1.5 -> lower=-0.05 upper=1.2 effort=10 velocity=1.5; mimic (none) -> joint=r_f_joint5_3 multiplier=0.9023 offset=-0.0410

File: scene/urdf/ur10_dexhand.urdf (robot description, URDF)
Before this commit: robot ur10_dexhand, 43 links, 42 joints
Joints:
- joint l_f_joint1_3: mimic joint=l_f_joint1_4 multiplier=1.0096 offset=0.0795 -> (none)
- joint l_f_joint1_4: limit lower=0 upper=1.3 effort=10 velocity=1.5 -> lower=-0.05 upper=1.2 effort=10 velocity=1.5; mimic (none) -> joint=l_f_joint1_3 multiplier=0.9023 offset=-0.0410
- joint l_f_joint2_3: mimic joint=l_f_joint2_4 multiplier=1.0096 offset=0.0795 -> (none)
- joint l_f_joint2_4: limit lower=0 upper=1.3 effort=10 velocity=1.5 -> lower=-0.05 upper=1.2 effort=10 velocity=1.5; mimic (none) -> joint=l_f_joint2_3 multiplier=0.9023 offset=-0.0410
- joint l_f_joint3_3: mimic joint=l_f_joint3_4 multiplier=1.0096 offset=0.0795 -> (none)
- joint l_f_joint3_4: limit lower=0 upper=1.3 effort=10 velocity=1.5 -> lower=-0.05 upper=1.2 effort=10 velocity=1.5; mimic (none) -> joint=l_f_joint3_3 multiplier=0.9023 offset=-0.0410
- joint l_f_joint4_3: mimic joint=l_f_joint4_4 multiplier=1.0096 offset=0.0795 -> (none)
- joint l_f_joint4_4: limit lower=0 upper=1.3 effort=10 velocity=1.5 -> lower=-0.05 upper=1.2 effort=10 velocity=1.5; mimic (none) -> joint=l_f_joint4_3 multiplier=0.9023 offset=-0.0410
- joint l_f_joint5_3: mimic joint=l_f_joint5_4 multiplier=1.0096 offset=0.0795 -> (none)
- joint l_f_joint5_4: limit lower=0 upper=1.3 effort=10 velocity=1.5 -> lower=-0.05 upper=1.2 effort=10 velocity=1.5; mimic (none) -> joint=l_f_joint5_3 multiplier=0.9023 offset=-0.0410
